File: ortholinear-keyboard/ortholinear-keyboard.sch (KiCad schematic (older format))
At the start: 136 parts, among them J1 USB, P1 TC2030-CTX-Tag-Connect, SW1 PG1353, SW10 PG1353, SW11 PG1353, SW12 PG1353, SW13 PG1353, SW14 PG1353, SW15 PG1353, SW16 PG1353, SW17 PG1353, SW18 PG1353, SW19 PG1353, SW2 PG1353, SW20 PG1353, SW21 PG1353, SW22 PG1353, SW23 PG1353, SW24 PG1353, SW25 PG1353, SW26 PG1353, SW27 PG1353, SW28 PG1353, SW29 PG1353, SW3 PG1353, SW30 PG1353, SW31 PG1353, SW32 PG1353, SW33 PG1353, SW34 PG1353, SW35 PG1353, SW36 PG1353, SW37 PG1353, SW38 PG1353, SW39 PG1353, SW4 PG1353, SW40 PG1353, SW41 PG1353, SW42 PG1353, SW43 PG1353, SW44 PG1353, SW45 PG1353, SW46 PG1353, SW47 PG1353, SW48 PG1353, SW49 PG1353, SW5 PG1353, SW50 PG1353, SW51 PG1353, SW52 PG1353, SW53 PG1353, SW54 PG1353, SW55 PG1353, SW56 PG1353, SW57 PG1353, SW58 PG1353, SW59 PG1353, SW6 PG1353, SW60 PG1353, SW7 PG1353, SW8 PG1353, SW9 PG1353, U1 STM32F042K6Ux, U2 XC6206PxxxMR

Commit message: exported production files
Parts:
- added D61: SP0502BAHT, Package_TO_SOT_SMD:SOT-23, symbol Power_Protection:SP0502BAHT
Connections:
- net C1: now also U1.11 (PA5); no longer U1.6 (PA0)
- net C10: now also U1.18 (PA8); no longer U1.19 (PA9)
- net C11: now also U1.13 (PA7); no longer U1.20 (PA10)
- net C12: now also U1.12 (PA6); no longer U1.25 (PA15)
- net C2: now also U1.10 (PA4); no longer U1.7 (PA1)
- net C3: now also U1.9 (PA3); no longer U1.8 (PA2)
- net C4: now also U1.8 (PA2); no longer U1.9 (PA3)
- net C5: now also U1.7 (PA1); no longer U1.10 (PA4)
- net C6: now also U1.6 (PA0); no longer U1.11 (PA5)
- net C7: now also U1.25 (PA15); no longer U1.12 (PA6)
- net C8: now also U1.20 (PA10); no longer U1.13 (PA7)
- net C9: now also U1.19 (PA9); no longer U1.18 (PA8)
- net D+: now also D61.1 (K)
- net D-: now also D61.2 (K)
- net GND: now also D61.3 (A)
- net R1: now also U1.32 (PB8); no longer U1.14 (PB0)
- net R2: now also U1.30 (PB7); no longer U1.15 (PB1)
- net R3: now also U1.29 (PB6); no longer U1.16 (PB2)
- net R4: now also U1.28 (PB5); no longer U1.26 (PB3)
Changed lines of the file:
@@
 Text GLabel 10400 800  1    50   Input ~ 0
 C12
+Text GLabel 2350 1800 2    50   Input ~ 0
+C1
+Text GLabel 2350 1700 2    50   Input ~ 0
+C2
+Text GLabel 2350 1600 2    50   Input ~ 0
+C3
+Text GLabel 2350 1500 2    50   Input ~ 0
+C4
+Text GLabel 2350 1400 2    50   Input ~ 0
+C5
 Text GLabel 2350 1300 2    50   Input ~ 0
-C1
-Text GLabel 2350 1400 2    50   Input ~ 0
-C2
-Text GLabel 2350 1500 2    50   Input ~ 0
-C3
-Text GLabel 2350 1600 2    50   Input ~ 0
-C4
-Text GLabel 2350 1700 2    50   Input ~ 0
-C5
-Text GLabel 2350 1800 2    50   Input ~ 0
 C6
+Text GLabel 2350 2800 2    50   Input ~ 0
+C7
+Text GLabel 2350 2300 2    50   Input ~ 0
+C8
+Text GLabel 2350 2200 2    50   Input ~ 0
+C9
+Text GLabel 2350 2100 2    50   Input ~ 0
+C10
+Text GLabel 2350 2000 2    50   Input ~ 0
+C11
 Text GLabel 2350 1900 2    50   Input ~ 0
-C7
-Text GLabel 2350 2000 2    50   Input ~ 0
-C8
-Text GLabel 2350 2100 2    50   Input ~ 0
-C9
-Text GLabel 2350 2200 2    50   Input ~ 0
-C10
-Text GLabel 2350 2300 2    50   Input ~ 0
-C11
-Text GLabel 2350 2800 2    50   Input ~ 0
 C12
-Text GLabel 1350 2000 0    50   Input ~ 0
+Text GLabel 1350 2800 0    50   Input ~ 0
 R1
-Text GLabel 1350 2100 0    50   Input ~ 0
+Text GLabel 1350 2700 0    50   Input ~ 0
 R2
-Text GLabel 1350 2200 0    50   Input ~ 0
+Text GLabel 1350 2600 0    50   Input ~ 0
 R3
-Text GLabel 1350 2300 0    50   Input ~ 0
+Text GLabel 1350 2500 0    50   Input ~ 0
 R4
 Text GLabel 1350 2400 0    50   Input ~ 0
@@
 	1    0    0    -1
 $EndComp
+$Comp
+L Power_Protection:SP0502BAHT D61
+U 1 1 60A63512
+P 2950 4450
+F 0 "D61" H 3155 4496 50  0000 L CNN
+F 1 "SP0502BAHT" H 3155 4405 50  0000 L CNN
+F 2 "Package_TO_SOT_SMD:SOT-23" H 3175 4400 50  0001 L CNN
+F 3 "http://www.littelfuse.com/~/media/files/littelfuse/technical%20resources/documents/data%20sheets/sp05xxba.pdf" H 3075 4575 50  0001 C CNN
+	1    2950 4450
+	1    0    0    -1
+$EndComp
+$Comp
+L power:GND #PWR0101
+U 1 1 60A63C4A
+P 2950 4650
+F 0 "#PWR0101" H 2950 4400 50  0001 C CNN
+F 1 "GND" H 2955 4477 50  0000 C CNN
+F 2 "" H 2950 4650 50  0001 C CNN
+F 3 "" H 2950 4650 50  0001 C CNN
+	1    2950 4650
+	1    0    0    -1
+$EndComp
+Text GLabel 3050 4250 1    50   Input ~ 0
+D-
+Text GLabel 2850 4250 1    50   Input ~ 0
+D+
 $EndSCHEMATC
